File: hardware/hardware_schematic.kicad_sch (KiCad schematic)
At the start: 8 parts, among them SW1 BUTTON, U1 TC1602A-01T, U2 DS18B20

Commit message: hw: correct schematic
Connections:
- net GND: no longer R2.1
- net at R1.1: now also SW1.2; no longer SW1.1
- net at A1.17 (D2): now also SW1.1; no longer SW1.2
- net at A1.18 (D3), U2.2 (DQ): now also R2.1
