File: hardware/hardware_schematic.kicad_sch (KiCad schematic)
At the start: 8 parts, among them SW1 BUTTON, U1 TC1602A-01T, U2 DS18B20

Commit message: hw: correct schematic
Parts:
- R1: value 1 kΩ -> 10 kΩ
- R2: value 1 kΩ -> 4.7 kΩ
- R3: value 1 kΩ -> 220 Ω
Changed lines of the file:
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@@
       (effects (font (size 1.27 1.27)) (justify left) hide)
     )
-    (property "Value" "1 kΩ" (at 128.27 121.92 0)
+    (property "Value" "4.7 kΩ" (at 128.27 121.92 0)
       (effects (font (size 1.27 1.27)) (justify left))
     )
@@
       (effects (font (size 1.27 1.27)) hide)
     )
-    (property "Value" "1 kΩ" (at 176.53 140.97 90)
+    (property "Value" "10 kΩ" (at 176.53 140.97 90)
       (effects (font (size 1.27 1.27)))
     )
@@
       (effects (font (size 1.27 1.27)) hide)
     )
-    (property "Value" "1 kΩ" (at 252.73 52.07 90)
+    (property "Value" "220 Ω" (at 252.73 52.07 90)
       (effects (font (size 1.27 1.27)))
     )

Commit message: hw: correct schematic
Connections:
- net at U1.11 (DB4): now also A1.28 (D13); no longer A1.25 (D10)
- net at U1.12 (DB5): now also A1.27 (D12); no longer A1.26 (D11)
- net at U1.13 (DB6): now also A1.26 (D11); no longer A1.27 (D12)
- net at U1.14 (DB7): now also A1.25 (D10); no longer A1.28 (D13)
