File: hardware/hardware.kicad_sch (KiCad schematic)
At the start: 8 parts, among them SW1 BUTTON, U1 TC1602A-01T, U2 DS18B20

Commit message: correct schematic
Connections:
- net +5V: now also SW1.1
- net at R1.1, SW1.2: now also A1.17 (D2)
